File: solderbit-segment-v0.1-SMT/solderbit-segment-v0.1-SMT.kicad_pcb (KiCad board)
At the start: 2 copper layers, 25 x 42 mm, 14 parts, among them J1 Conn_01x05_Pin, U2 PCF8574N

Commit message: Separate SMT version, and THT I/O expander
Parts:
- removed U2: PCF8574N, SolderbitSegment:DIP-16
- added U1: PCF8574AT, SolderbitSegment:SO-16, F.Cu at (140.0, 78.0)
- C1: value 1uF -> C_Small
- moved C1 19.5 mm to (149.0, 75.9), turned to -90 degrees
- moved R5 12.1 mm to (149.0, 102.4)
- moved R8 11.9 mm to (149.0, 90.4)
- moved G*** 4.50 mm to (140.0, 87.5)
- moved R6 4.06 mm to (149.0, 98.4)
- moved R7 3.94 mm to (149.0, 94.4)
Routing:
- net /P7: track 36.0 -> 15.2 mm
- net GND: track 0.00 -> 17.5 mm, vias 17 -> 18
- net Net-(DS1-D.P.): track 3.94 -> 17.1 mm
- net /P6: track 29.9 -> 18.0 mm
- net /P3: track 33.8 -> 23.1 mm
- net /P2: track 27.6 -> 20.4 mm
- net /~{INT}: track 7.22 -> 13.3 mm
- net /SDA: track 15.8 -> 10.5 mm
- net Net-(DS1-G): track 25.5 -> 20.2 mm
- net /P4: track 18.8 -> 23.9 mm
- net Net-(DS1-F): track 17.6 -> 22.4 mm
- net Net-(DS1-E): track 19.6 -> 15.1 mm, vias 2 -> 0
- net /P5: track 23.8 -> 20.7 mm
- net /P1: track 21.7 -> 19.2 mm
- net Net-(DS1-D): track 9.65 -> 7.51 mm
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